File: LED_FAN_CONTROLLER/LED_FAN_CONTROLLER.kicad_sch (KiCad schematic)
At the start: 21 parts, among them J2 Barrel_Jack, J3 Conn_01x04, J4 Conn_01x04, J5 Conn_01x07_MountingPin, Q2 IRLL014TRPBF, Q3 IRLL014TRPBF, Q4 IRLL014TRPBF, Q5 IRLL014TRPBF, U1 MIC5231-3.3YM5-TR, U2 MC74HC1G04DFT2

Commit message: Add files via upload
Parts:
- removed U2: MC74HC1G04DFT2, Package_TO_SOT_SMD:SOT-353_SC-70-5, symbol Power_Management:FPF2002
- added U4: MC74HC1G04DFT2G, SC70-5_ONS, symbol 2024-08-03_19-30-19:MC74HC1G04DFT2G
Connections:
- net at J2.2, J5.7 (Pin_7), Q2.3 (S)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: now also U4.3 (GND)
- net at R13.1, U1.5 (VOUT): now also U4.5 (VCC)
- net at R2.2: now also U4.2 (INA)
- net at J4.4 (Pin_4): now also U4.4 (OUT*Y)
Changed lines of the file:
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@@
   (junction (at 149.86 100.33) (diameter 0) (color 0 0 0 1)
   )
+  (junction (at 170.18 49.53) (diameter 0) (color 255 255 0 1)
+  )
   (junction (at 91.44 64.77) (diameter 0) (color 0 0 0 1)
   )
@@
   (junction (at 104.14 49.53) (diameter 0) (color 255 0 0 1)
   )
+  (junction (at 179.07 78.74) (diameter 0) (color 0 0 0 1)
+  )
   (junction (at 161.29 115.57) (diameter 0) (color 0 0 0 0)
   )
@@
   (junction (at 161.29 129.54) (diameter 0) (color 0 0 0 0)
   )
-  (junction (at 170.18 49.53) (diameter 0) (color 255 255 0 1)
-  )
   (junction (at 149.86 137.16) (diameter 0) (color 0 0 0 1)
   )
   (junction (at 161.29 143.51) (diameter 0) (color 0 0 0 0)
   )
-  (junction (at 179.07 78.74) (diameter 0) (color 0 0 0 1)
-  )
   (wire (pts (xy 160.02 73.66) (xy 170.18 73.66))
     (stroke (width 0) (type default))
@@
   )
   (wire (pts (xy 189.23 152.4) (xy 189.23 148.59))
+    (stroke (width 0) (type default) (color 0 0 0 1))
+  )
+  (wire (pts (xy 220.98 102.87) (xy 179.07 102.87))
     (stroke (width 0) (type default) (color 0 0 0 1))
   )
@@
     (stroke (width 0) (type default) (color 255 255 0 1))
   )
+  (wire (pts (xy 220.98 91.44) (xy 220.98 49.53))
+    (stroke (width 0) (type default) (color 255 255 0 1))
+  )
   (wire (pts (xy 104.14 49.53) (xy 133.35 49.53))
     (stroke (width 0) (type default) (color 255 0 0 1))
@@
     (stroke (width 0) (type default) (color 0 0 0 1))
   )
-  (wire (pts (xy 201.93 99.06) (xy 208.28 99.06))
-    (stroke (width 0) (type default) (color 255 255 0 1))
-  )
   (wire (pts (xy 160.02 64.77) (xy 179.07 64.77))
     (stroke (width 0) (type default) (color 0 0 0 1))
   )
-  (wire (pts (xy 176.53 87.63) (xy 191.77 87.63))
-    (stroke (width 0) (type default))
-  )
   (wire (pts (xy 91.44 54.61) (xy 88.9 54.61))
-    (stroke (width 0) (type default) (color 0 0 0 1))
-  )
-  (wire (pts (xy 181.61 93.98) (xy 179.07 93.98))
     (stroke (width 0) (type default) (color 0 0 0 1))
   )
@@
     (stroke (width 0) (type default))
   )
+  (wire (pts (xy 220.98 93.98) (xy 222.25 93.98))
+    (stroke (width 0) (type default) (color 19 0 255 1))
+  )
   (wire (pts (xy 175.26 129.54) (xy 181.61 129.54))
     (stroke (width 0) (type default))
@@
     (stroke (width 0) (type default) (color 255 0 0 1))
   )
-  (wire (pts (xy 170.18 49.53) (xy 208.28 49.53))
+  (wire (pts (xy 156.21 85.09) (xy 193.04 85.09))
+    (stroke (width 0) (type default) (color 255 0 0 1))
+  )
+  (wire (pts (xy 205.74 138.43) (xy 189.23 138.43))
+    (stroke (width 0) (type default))
+  )
+  (wire (pts (xy 199.39 73.66) (xy 229.87 73.66))
+    (stroke (width 0) (type default))
+  )
+  (wire (pts (xy 158.75 87.63) (xy 163.83 87.63))
+    (stroke (width 0) (type default))
+  )
+  (wire (pts (xy 170.18 49.53) (xy 220.98 49.53))
     (stroke (width 0) (type default) (color 255 255 0 1))
   )
-  (wire (pts (xy 156.21 85.09) (xy 193.04 85.09))
-    (stroke (width 0) (type default) (color 255 0 0 1))
-  )
-  (wire (pts (xy 205.74 138.43) (xy 189.23 138.43))
-    (stroke (width 0) (type default))
-  )
-  (wire (pts (xy 199.39 73.66) (xy 229.87 73.66))
-    (stroke (width 0) (type default))
-  )
-  (wire (pts (xy 158.75 87.63) (xy 163.83 87.63))
-    (stroke (width 0) (type default))
-  )
   (wire (pts (xy 153.67 73.66) (xy 160.02 73.66))
     (stroke (width 0) (type default))
   )
+  (wire (pts (xy 222.25 76.2) (xy 229.87 76.2))
+    (stroke (width 0) (type default) (color 0 0 255 1))
+  )
   (wire (pts (xy 193.04 71.12) (xy 229.87 71.12))
     (stroke (width 0) (type default) (color 255 0 0 1))
@@
     (stroke (width 0) (type default))
   )
-  (wire (pts (xy 208.28 49.53) (xy 208.28 99.06))
-    (stroke (width 0) (type default) (color 255 255 0 1))
+  (wire (pts (xy 220.98 96.52) (xy 220.98 102.87))
+    (stroke (width 0) (type default) (color 0 0 0 1))
+  )
+  (wire (pts (xy 179.07 102.87) (xy 179.07 78.74))
+    (stroke (width 0) (type default) (color 0 0 0 1))
   )
   (wire (pts (xy 189.23 68.58) (xy 229.87 68.58))
@@
     (stroke (width 0) (type default) (color 0 0 0 1))
   )
+  (wire (pts (xy 176.53 87.63) (xy 176.53 93.98))
+    (stroke (width 0) (type default))
+  )
   (wire (pts (xy 229.87 109.22) (xy 200.66 109.22))
     (stroke (width 0) (type default))
@@
     (stroke (width 0) (type default) (color 0 0 0 1))
   )
-  (wire (pts (xy 203.2 76.2) (xy 229.87 76.2))
-    (stroke (width 0) (type default) (color 0 0 255 1))
+  (wire (pts (xy 222.25 93.98) (xy 222.25 76.2))
+    (stroke (width 0) (type default) (color 19 0 255 1))
   )
   (wire (pts (xy 139.7 129.54) (xy 139.7 118.11))
@@
     (stroke (width 0) (type default) (color 255 255 0 1))
   )
+  (wire (pts (xy 176.53 93.98) (xy 180.34 93.98))
+    (stroke (width 0) (type default))
+  )
   (wire (pts (xy 91.44 64.77) (xy 91.44 100.33))
     (stroke (width 0) (type default) (color 0 0 0 1))
@@
     (stroke (width 0) (type default))
   )
-  (wire (pts (xy 201.93 93.98) (xy 203.2 93.98))
-    (stroke (width 0) (type default) (color 0 0 255 1))
-  )
   (wire (pts (xy 153.67 107.95) (xy 91.44 107.95))
     (stroke (width 0) (type default))
@@
     (stroke (width 0) (type default))
   )
-  (wire (pts (xy 203.2 76.2) (xy 203.2 93.98))
-    (stroke (width 0) (type default) (color 0 0 255 1))
-  )
   (wire (pts (xy 91.44 132.08) (xy 81.28 132.08))
     (stroke (width 0) (type default) (color 0 0 0 1))
@@
   )
   (wire (pts (xy 149.86 100.33) (xy 149.86 123.19))
-    (stroke (width 0) (type default) (color 0 0 0 1))
-  )
-  (wire (pts (xy 179.07 78.74) (xy 179.07 93.98))
     (stroke (width 0) (type default) (color 0 0 0 1))
   )
@@
     (stroke (width 0) (type default) (color 255 255 0 1))
   )
-  (wire (pts (xy 191.77 87.63) (xy 191.77 88.9))
-    (stroke (width 0) (type default))
-  )
   (wire (pts (xy 200.66 109.22) (xy 200.66 124.46))
     (stroke (width 0) (type default))
@@
         (path "/b877c464-db5e-4743-8cb3-a02e326c6afa"
           (reference "J2") (unit 1)
-        )
-      )
-    )
-  )
-  (symbol (lib_id "Power_Management:FPF2002") (at 191.77 96.52 180) (unit 1)
-    (in_bom yes) (on_board yes) (dnp no) (fields_autoplaced)
-    (property "Reference" "U2" (at 191.77 104.14 0)
-      (effects (font (size 1.27 1.27)))
-    )
-    (property "Value" "MC74HC1G04DFT2" (at 191.77 106.68 0)
-      (effects (font (size 1.27 1.27)))
-    )
-    (property "Footprint" "Package_TO_SOT_SMD:SOT-353_SC-70-5" (at 168.91 88.9 0)
-      (effects (font (size 1.27 1.27)) hide)
-    )
-    (property "Datasheet" "https://www.onsemi.com/pub/Collateral/FPF2001-D.pdf" (at 193.04 106.68 0)
-      (effects (font (size 1.27 1.27)) hide)
-    )
-    (pin "3")
-    (pin "1")
-    (pin "2")
-    (pin "4")
-    (pin "5")
-    (instances
-      (project "LED_FAN_CONTROLLER"
-        (path "/b877c464-db5e-4743-8cb3-a02e326c6afa"
-          (reference "U2") (unit 1)
         )
       )
@@
         )
       )
+    )
+  )
+  (symbol (lib_id "2024-08-03_19-30-19:MC74HC1G04DFT2G") (at 180.34 91.44 0) (unit 1)
+    (in_bom yes) (on_board yes) (dnp no) (fields_autoplaced)
+    (property "Reference" "U4" (at 200.66 81.28 0)
+      (effects (font (size 1.524 1.524)))
+    )
+    (property "Value" "MC74HC1G04DFT2G" (at 200.66 83.82 0)
+      (effects (font (size 1.524 1.524)))
+    )
+    (property "Footprint" "SC70-5_ONS" (at 180.34 91.44 0)
+      (effects (font (size 1.27 1.27) italic) hide)
+    )
+    (property "Datasheet" "MC74HC1G04DFT2G" (at 180.34 91.44 0)
+      (effects (font (size 1.27 1.27) italic) hide)
+    )
+    (pin "5")
+    (pin "4")
+    (pin "1")
+    (pin "3")
+    (pin "2")
+    (instances
+      (project "LED_FAN_CONTROLLER"
+        (path "/b877c464-db5e-4743-8cb3-a02e326c6afa"
+          (reference "U4") (unit 1)
+        )
+      )
