File: LED_FAN_CONTROLLER/LED_FAN_CONTROLLER.kicad_pcb (KiCad board)
At the start: 2 copper layers, 42 x 41.3 mm, 22 parts, among them J2 Barrel_Jack, J3 Conn_01x04, J4 Conn_01x04, J5 Conn_01x07_MountingPin, Q2 IRLL014TRPBF, Q3 IRLL014TRPBF, Q4 IRLL014TRPBF, Q5 IRLL014TRPBF, U1 MIC5231-5.0YM5-TR, U2 MC74HC1G04DFT2

Commit message: Add files via upload
Parts:
- added R13: 10000, Resistor_SMD:R_0603_1608Metric, F.Cu at (148.9, 91.4)
- U1: value MIC5231-5.0YM5-TR -> MIC5231-3.3YM5-TR
Connections:
- R2 pad 2: Net-(U2-GND) -> Net-(U4-INA)
Routing:
- net Net-(U2-GND): track 9.66 -> 0.00 mm
- net Net-(U1-VOUT): track 14.1 -> 16.5 mm
- net Net-(J4-Pin_3): track 41.9 -> 43.6 mm
